File: light-atreus.sch (KiCad schematic (older format))
At the start: 11 parts, among them J1 USB_B, J10 CONN_01X02, J11 USB_B, J2 CONN_01X02, J3 CONN_01X02, J4 CONN_01X02, J5 CONN_01X02, J6 CONN_01X02, J7 CONN_01X02, J8 CONN_01X02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

Commit message: Add names to all important nets
Connections:
- net labels added: D+, D-, SHIELD
Changed lines of the file:
@@
 	5850 5100 5850 4450
 Connection ~ 5850 4450
+Text Label 3950 4450 0    60   ~ 0
+SHIELD
+Text Label 4350 3850 0    60   ~ 0
+D+
+Text Label 4200 3950 0    60   ~ 0
+D-
 $EndSCHEMATC

Commit message: Remove shield wire solder point breakout
Parts:
- removed J10: CONN_01X02, custom_footprints:SolderWirePad_1x2-8mm, symbol CONN_01X02
Connections:
- wire segments 23 -> 21
- no-connect marks 9 -> 8
Changed lines of the file:
@@
-$EndComp
-$Comp
-L CONN_01X02 J10
-U 1 1 59CD667D
-P 6300 5150
-F 0 "J10" H 6218 4875 50  0000 C CNN
-F 1 "CONN_01X02" H 6218 4966 50  0000 C CNN
-F 2 "custom_footprints:SolderWirePad_1x2-8mm" H 6300 5150 50  0001 C CNN
-F 3 "" H 6300 5150 50  0001 C CNN
-	1    6300 5150
-	1    0    0    -1
 $EndComp
 $Comp
@@
 NoConn ~ 6100 2200
 NoConn ~ 6100 4750
-NoConn ~ 6100 5200
 Wire Wire Line
 	6100 4650 5950 4650
@@
 	5950 4650 5950 4350
 Connection ~ 5950 4350
-Wire Wire Line
-	6100 5100 5850 5100
-Wire Wire Line
-	5850 5100 5850 4450
-Connection ~ 5850 4450
 Text Label 3950 4450 0    60   ~ 0
 SHIELD
